File: hardware/bleezy.kicad_pcb (KiCad board)
At the start: 2 copper layers, 65 x 30 mm, 46 parts, among them IC1 NRF51822, P1 Analog Header, P2 Digital Con 2, P3 Raspberry_Pi_+_Conn, P5 Power Con, P6 TST, Q1 BSS138, U1 LD3985M33R, U5 DMMT5401, Y1 32Khz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

Commit message: changed some silk labels
Routing:
- net (no net): track 0.00 -> 2.00 mm
- net GND: track 74.3 -> 72.3 mm
Other:
- board text added: "nRF Connections"
Changed lines of the file:
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@@
-(kicad_pcb (version 4) (host pcbnew 4.0.1-stable)
+(kicad_pcb (version 4) (host pcbnew 4.0.1-3.201512221402+6198~38~ubuntu14.04.1-stable)
   (general
     (links 118)
@@
     (area 35.49 14.500001 119.679167 72.1685)
     (thickness 1.6)
-    (drawings 61)
+    (drawings 64)
     (tracks 650)
     (zones 0)
@@
     )
   )
+  (gr_line (start 73.4 54) (end 62.5 54) (layer B.SilkS) (width 0.35))
+  (gr_text "nRF Connections" (at 73.7 53) (layer B.SilkS)
+    (effects (font (size 0.9 0.9) (thickness 0.2)) (justify left mirror))
+  )
+  (gr_line (start 92.4 69.2) (end 92.4 59) (layer B.SilkS) (width 0.35))
   (gr_line (start 102.6 45.7) (end 102.6 43.2) (layer F.SilkS) (width 0.35))
   (gr_line (start 96.6 45.7) (end 102.6 45.7) (layer F.SilkS) (width 0.35))
@@
     (effects (font (size 0.7 0.7) (thickness 0.175)))
   )
-  (gr_text "PI Connections\nGPIO14>P09\nGPIO15>P10\nGPIO10>P11\nGPIO09>P12\nGPIO11>P13\nGPIO08>P14\nGPIO05>P07\nGPIO06>P08" (at 85.7 69.2 270) (layer B.SilkS)
-    (effects (font (size 0.7 0.7) (thickness 0.175)) (justify left mirror))
+  (gr_text "PI Connections\n\nGPIO14>P09\nGPIO15>P10\nGPIO10>P11\nGPIO09>P12\nGPIO11>P13\nGPIO08>P14\nGPIO05>P07\nGPIO06>P08" (at 87.3 69.2 270) (layer B.SilkS)
+    (effects (font (size 0.9 0.9) (thickness 0.2)) (justify left mirror))
   )
   (gr_text "5V\nVCC\nGND\nGND" (at 98.5 54.5) (layer F.SilkS)
     (effects (font (size 1 1) (thickness 0.25)))
   )
-  (gr_line (start 80.95 52.977866) (end 89.95 52.977866) (layer B.SilkS) (width 0.2))
-  (gr_line (start 80.95 49.977866) (end 80.95 52.977866) (layer B.SilkS) (width 0.2))
-  (gr_line (start 89.95 49.977866) (end 80.95 49.977866) (layer B.SilkS) (width 0.2))
-  (gr_arc (start 89.95 51.477866) (end 89.95 52.977866) (angle -180) (layer B.SilkS) (width 0.2))
-  (gr_line (start 80.95 56.959754) (end 89.95 56.959754) (layer B.SilkS) (width 0.2))
-  (gr_line (start 80.95 53.959754) (end 80.95 56.959754) (layer B.SilkS) (width 0.2))
-  (gr_line (start 89.95 53.959754) (end 80.95 53.959754) (layer B.SilkS) (width 0.2))
-  (gr_arc (start 89.95 55.459754) (end 89.95 56.959754) (angle -180) (layer B.SilkS) (width 0.2))
-  (gr_text P2 (at 90.15 51.477866 270) (layer B.SilkS)
+  (gr_line (start 62.75 58.977866) (end 71.75 58.977866) (layer B.SilkS) (width 0.2))
+  (gr_line (start 62.75 55.977866) (end 62.75 58.977866) (layer B.SilkS) (width 0.2))
+  (gr_line (start 71.75 55.977866) (end 62.75 55.977866) (layer B.SilkS) (width 0.2))
+  (gr_arc (start 71.75 57.477866) (end 71.75 58.977866) (angle -180) (layer B.SilkS) (width 0.2))
+  (gr_line (start 62.75 62.959754) (end 71.75 62.959754) (layer B.SilkS) (width 0.2))
+  (gr_line (start 62.75 59.959754) (end 62.75 62.959754) (layer B.SilkS) (width 0.2))
+  (gr_line (start 71.75 59.959754) (end 62.75 59.959754) (layer B.SilkS) (width 0.2))
+  (gr_arc (start 71.75 61.459754) (end 71.75 62.959754) (angle -180) (layer B.SilkS) (width 0.2))
+  (gr_text P2 (at 71.95 57.477866 270) (layer B.SilkS)
     (effects (font (size 1 1) (thickness 0.25)) (justify mirror))
   )
-  (gr_text P1 (at 90.15 55.459754 270) (layer B.SilkS)
+  (gr_text P1 (at 71.95 61.459754 270) (layer B.SilkS)
     (effects (font (size 1 1) (thickness 0.25)) (justify mirror))
   )
-  (gr_text "P0.15\nP0.16\nP0.17\nP0.18\nP0.19\nP0.20\nP0.21\nP0.22" (at 85.05 51.477866 270) (layer B.SilkS)
+  (gr_text "P0.15\nP0.16\nP0.17\nP0.18\nP0.19\nP0.20\nP0.21\nP0.22" (at 66.85 57.477866 270) (layer B.SilkS)
     (effects (font (size 0.6 0.6) (thickness 0.15)) (justify mirror))
   )
-  (gr_text "P0.00\nP0.01\nP0.02\nP0.03\nP0.04\nP0.05\nP0.06\nGND" (at 85.05 55.459754 270) (layer B.SilkS)
+  (gr_text "P0.00\nP0.01\nP0.02\nP0.03\nP0.04\nP0.05\nP0.06\nGND" (at 66.85 61.459754 270) (layer B.SilkS)
     (effects (font (size 0.6 0.6) (thickness 0.15)) (justify mirror))
   )
@@
   )
   (gr_arc (start 41.1 42.7) (end 38.1 42.7) (angle 90) (layer Edge.Cuts) (width 0.1))
+  (segment (start 52.85 55.157107) (end 52.142893 54.45) (width 0.5) (layer B.Cu) (net 0))
+  (segment (start 53.557107 55.864214) (end 54.264214 55.157107) (width 0.5) (layer B.Cu) (net 0))
   (segment (start 101.5 55.77) (end 101.5 58.31) (width 0.3) (layer F.Cu) (net 1))
   (segment (start 53.612947 62.437947) (end 53.29528 62.755614) (width 0.2) (layer F.Cu) (net 1))
@@
   (segment (start 52.85 55.157107) (end 52.142893 55.864214) (width 0.5) (layer F.Cu) (net 1))
   (segment (start 52.142893 54.45) (end 51.435786 55.157107) (width 0.5) (layer F.Cu) (net 1))
-  (segment (start 52.85 55.157107) (end 52.142893 54.45) (width 0.5) (layer B.Cu) (net 1))
   (segment (start 53.557107 54.45) (end 52.85 55.157107) (width 0.5) (layer F.Cu) (net 1))
   (segment (start 52.85 52.32868) (end 52.142893 53.035786) (width 0.5) (layer F.Cu) (net 1))
@@
   (segment (start 53.557107 54.45) (end 54.264214 53.742893) (width 0.5) (layer B.Cu) (net 1))
   (segment (start 54.264214 55.157107) (end 53.557107 54.45) (width 0.5) (layer F.Cu) (net 1))
-  (segment (start 53.557107 55.864214) (end 54.264214 55.157107) (width 0.5) (layer B.Cu) (net 1))
   (segment (start 52.85 56.57132) (end 53.557107 55.864214) (width 0.5) (layer F.Cu) (net 1))
   (segment (start 50.72868 54.45) (end 52.85 56.57132) (width 0.5) (layer B.Cu) (net 1))
